Commit message: Added sensor links to URDF

File: earthrovers_description/src/description/frodobot.urdf (robot description, URDF)
Before this commit: robot rover, 2 links, 1 joints
Links:
- added link front_camera_link; visual box size=0.05 0.05 0.05
- added link imu_link; visual box size=0.05 0.05 0.05
- added link rear_camera_link; visual box size=0.05 0.05 0.05
Joints:
- added joint front_camera_joint: type fixed, parent base_link, child front_camera_link, origin xyz=0.013 0.0 0.561 rpy=0 0 0
- added joint imu_joint: type fixed, parent base_link, child imu_link, origin xyz=0.0 0.0 0.561 rpy=0 0 0
- added joint rear_camera_joint: type fixed, parent base_link, child rear_camera_link, origin xyz=0.0 0.0 0.561 rpy=0 0 3.14

Commit message: Added gps_link

File: earthrovers_description/src/description/frodobot.urdf (robot description, URDF)
Before this commit: robot rover, 5 links, 4 joints
Links:
- added link gps_link; visual box size=0.05 0.05 0.05
Joints:
- added joint gps_joint: type fixed, parent base_link, child gps_link, origin xyz=0.0 0.0 0.0 rpy=0 0 0
